Commit message: [feature] Add UR10e meshes and start base_link STL integration (WIP)

File: src/robot_description/urdf/ur10e.urdf.xacro (robot description, xacro)
@@ -26,16 +26,4 @@
        Macros
        =============================== -->
-  <!-- Simple visual link (cylinder) -->
-  <xacro:macro name="simple_link" params="name length radius">
-    <link name="${name}">
-      <visual>
-        <!-- Cylinder axis is Z (원통 축은 Z) -->
-        <origin xyz="0 0 ${length/2.0}" rpy="0 0 0"/>
-        <geometry>
-          <cylinder length="${length}" radius="${radius}"/>
-        </geometry>
-      </visual>
-    </link>
-  </xacro:macro>
   <!-- Revolute joint from Classic DH -->
   <xacro:macro name="dh_revolute" params="name parent child a d alpha">
@@ -53,11 +41,19 @@
        Links
        =============================== -->
-  <xacro:simple_link name="base_link" length="0.05" radius="0.06"/>
-  <xacro:simple_link name="link1" length="0.10" radius="0.04"/>
-  <xacro:simple_link name="link2" length="0.10" radius="0.03"/>
-  <xacro:simple_link name="link3" length="0.10" radius="0.03"/>
-  <xacro:simple_link name="link4" length="0.08" radius="0.025"/>
-  <xacro:simple_link name="link5" length="0.08" radius="0.02"/>
-  <xacro:simple_link name="link6" length="0.06" radius="0.02"/>
+  <link name="base_link">
+    <visual>
+      <origin xyz="0 0 0" rpy="0 0 0"/>
+      <geometry>
+        <mesh filename="package://robot_description/meshes/base_link.STL"
+              scale="1 1 1"/>
+      </geometry>
+    </visual>
+  </link>
+  <link name="link1"/>
+  <link name="link2"/>
+  <link name="link3"/>
+  <link name="link4"/>
+  <link name="link5"/>
+  <link name="link6"/>
   <!-- ===============================
        Joints (Skeleton)

Commit message: [feature] Complete UR10e DH-to-URDF conversion
- Add detailed DH-to-URDF conversion strategy documentation
- Explain how to split DH joints into URDF joint pairs for correct transformation order
- Update roadmap to mark UR10e model alignment as complete

File: src/robot_description/urdf/ur10e.urdf.xacro (robot description, xacro)
@@ -1,85 +1,206 @@
 <?xml version="1.0"?>
 <robot name="robot_kinematics_sandbox" xmlns:xacro="http://www.ros.org/wiki/xacro">
+  <!-- =========================================================
+       What this file does (이 파일이 하는 일)
+       - UR10e의 Classic DH 파라미터를 그대로 사용
+       - URDF의 제약 때문에 DH 조인트 1개를 URDF 조인트 2개로 분리
+       - 수학적 기구학(DH)과 시각화(mesh 정렬)를 분리
+       핵심 아이디어:
+       DH의 회전/이동 순서를 URDF에서도 똑같이 만들기 위함
+       ========================================================= -->
+  <!-- =========================================================
+       DH 파라미터를 분리하여 URDF에 적용하는 이유
+       Classic DH 한 조인트의 순서:
+         1) z축으로 d 이동  (Trans(z, d))
+         2) z축 기준 θ 회전 (Rot(z, θ))
+         3) x축으로 a 이동  (Trans(x, a))
+         4) x축 기준 α 회전 (Rot(x, α))
+       하지만 URDF는:
+         - joint origin을 먼저 적용 (Trans))
+         - 그 다음에 joint 회전을 적용 (Rot))
+       그래서 a, d, α를 한 origin에 넣으면
+       α 회전이 θ보다 먼저 적용되어 회전축이 틀어진다.
+       해결 방법:
+         DH 조인트 1개를 URDF 조인트 2개로 분리
+       ========================================================= -->
+  <!-- =========================================================
+       DH → URDF conversion strategy (변환 전략)
+       parent
+         └─ revolute joint
+             - z축으로 d 이동 (Trans(z, d))
+             - z축 기준 θ 회전 (Rot(z, θ))
+         └─ virtual link (중간 프레임, 실제 로봇에는 없음)
+         └─ fixed joint
+             - x축으로 a 이동 (Trans(x, a))
+             - x축 기준 α 회전 (Rot(x, α))
+         └─ child
+       이렇게 하면 DH와 동일한 변환 순서 유지
+       Trans(z,d) → Rot(z,θ) → Trans(x,a) → Rot(x,α)
+       ========================================================= -->
   <!-- ===============================
-       DH parameters (Classic DH)
+       DH parameters for UR10e
        units: meter, radian
        =============================== -->
-  <xacro:property name="a1" value="0.0"/>
-  <xacro:property name="d1" value="0.1807"/>
+  <xacro:property name="a1"     value="0.0"/>
+  <xacro:property name="d1"     value="0.1807"/>
   <xacro:property name="alpha1" value="${pi/2}"/>
-  <xacro:property name="a2" value="-0.6127"/>
-  <xacro:property name="d2" value="0.0"/>
+  <xacro:property name="a2"     value="-0.6127"/>
+  <xacro:property name="d2"     value="0.0"/>
   <xacro:property name="alpha2" value="0.0"/>
-  <xacro:property name="a3" value="-0.57155"/>
-  <xacro:property name="d3" value="0.0"/>
+  <xacro:property name="a3"     value="-0.57155"/>
+  <xacro:property name="d3"     value="0.0"/>
   <xacro:property name="alpha3" value="0.0"/>
-  <xacro:property name="a4" value="0.0"/>
-  <xacro:property name="d4" value="0.17415"/>
+  <xacro:property name="a4"     value="0.0"/>
+  <xacro:property name="d4"     value="0.17415"/>
   <xacro:property name="alpha4" value="${pi/2}"/>
-  <xacro:property name="a5" value="0.0"/>
-  <xacro:property name="d5" value="0.11985"/>
+  <xacro:property name="a5"     value="0.0"/>
+  <xacro:property name="d5"     value="0.11985"/>
   <xacro:property name="alpha5" value="${-pi/2}"/>
-  <xacro:property name="a6" value="0.0"/>
-  <xacro:property name="d6" value="0.11655"/>
+  <xacro:property name="a6"     value="0.0"/>
+  <xacro:property name="d6"     value="0.11655"/>
   <xacro:property name="alpha6" value="0.0"/>
   <!-- ===============================
-       Macros
+       Macro: Classic DH → URDF
        =============================== -->
-  <!-- Revolute joint from Classic DH -->
   <xacro:macro name="dh_revolute" params="name parent child a d alpha">
+    <!-- 1) Revolute joint
+         - parent 기준 z축으로 d 이동
+         - z축 기준으로 θ 회전 -->
     <joint name="${name}" type="revolute">
       <parent link="${parent}"/>
-      <child link="${child}"/>
-      <!-- Classic DH: xyz=[a,0,d], rpy=[alpha,0,0] -->
-      <origin xyz="${a} 0 ${d}" rpy="${alpha} 0 0"/>
+      <child  link="${name}_virtual"/>
+      <origin xyz="0 0 ${d}" rpy="0 0 0"/>
       <axis xyz="0 0 1"/>
-      <!-- Visualization limits -->
       <limit lower="-6.283" upper="6.283" effort="200" velocity="3.0"/>
     </joint>
+    <!-- 2) Virtual link (기구학 계산용, 시각화 없음) -->
+    <link name="${name}_virtual"/>
+    <!-- 3) Fixed joint
+         - x축으로 a 이동
+         - x축 기준으로 α 회전 -->
+    <joint name="${name}_fixed" type="fixed">
+      <parent link="${name}_virtual"/>
+      <child  link="${child}"/>
+      <origin xyz="${a} 0 0" rpy="${alpha} 0 0"/>
+    </joint>
   </xacro:macro>
-  <!-- ===============================
-       Links
-       =============================== -->
+  <!-- =========================================================
+       Links and visual meshes
+       중요 원칙:
+       - joint / DH 파라미터는 "기구학"
+       - visual origin은 "메쉬 정렬"
+       - 메쉬 보정은 FK/IK에 영향 없음
+       ========================================================= -->
+  <!-- Base link -->
   <link name="base_link">
     <visual>
       <origin xyz="0 0 0" rpy="0 0 0"/>
       <geometry>
-        <mesh filename="package://robot_description/meshes/base_link.STL"
-              scale="1 1 1"/>
-      </geometry>
-    </visual>
-  </link>
-  <link name="link1"/>
-  <link name="link2"/>
-  <link name="link3"/>
-  <link name="link4"/>
-  <link name="link5"/>
-  <link name="link6"/>
-  <!-- ===============================
-       Joints (Skeleton)
-       =============================== -->
-  <xacro:dh_revolute name="shoulder_pan_joint"
+        <mesh filename="package://robot_description/meshes/base_link.dae"
+              scale="1 1 1"/>
+      </geometry>
+    </visual>
+  </link>
+  <!-- Link 1: Shoulder -->
+  <link name="link1">
+    <visual>
+      <origin xyz="0 0 0" rpy="-1.5708 -3.14159 0"/>
+      <geometry>
+        <mesh filename="package://robot_description/meshes/link1.dae"
+              scale="1 1 1"/>
+      </geometry>
+    </visual>
+  </link>
+  <!-- Link 2: Upper Arm -->
+  <link name="link2">
+    <visual>
+      <origin xyz="0.6127 0 0.1762" rpy="1.5708 0 -1.5708"/>
+      <geometry>
+        <mesh filename="package://robot_description/meshes/link2.dae"
+              scale="1 1 1"/>
+      </geometry>
+    </visual>
+  </link>
+  <!-- Link 3: Forearm -->
+  <link name="link3">
+    <visual>
+      <origin xyz="0.57155 0 0.0393" rpy="1.5708 0 -1.5708"/>
+      <geometry>
+        <mesh filename="package://robot_description/meshes/link3.dae"
+              scale="1 1 1"/>
+      </geometry>
+    </visual>
+  </link>
+  <!-- Link 4: Wrist 1 -->
+  <link name="link4">
+    <visual>
+      <origin xyz="0 -0.135 0" rpy="0 0 0"/>
+      <geometry>
+        <mesh filename="package://robot_description/meshes/link4.dae"
+              scale="1 1 1"/>
+      </geometry>
+    </visual>
+  </link>
+  <!-- Link 5: Wrist 2 -->
+  <link name="link5">
+    <visual>
+      <origin xyz="0 0.12 0" rpy="1.5708 0 0"/>
+      <geometry>
+        <mesh filename="package://robot_description/meshes/link5.dae"
+              scale="1 1 1"/>
+      </geometry>
+    </visual>
+  </link>
+  <!-- Link 6: Wrist 3 / Tool Flange -->
+  <link name="link6">
+    <visual>
+      <origin xyz="0 0 -0.1168" rpy="1.5708 0 0"/>
+      <geometry>
+        <mesh filename="package://robot_description/meshes/link6.dae"
+              scale="1 1 1"/>
+      </geometry>
+    </visual>
+  </link>
+  <!-- =========================================================
+     Joint structure (DH → URDF mapping)
+     Each DH joint is split into:
+       - revolute joint : d, θ
+       - fixed joint    : a, α
+       - virtual link   : frame separation only
+     Reason:
+       URDF applies joint origin before rotation,
+       so DH order must be preserved manually.
+     Kinematic chain:
+       base_link → link1 → link2 → link3 → link4 → link5 → link6 → tool0
+     ========================================================= -->
+  <!-- Joint 1: Shoulder Pan -->
+  <xacro:dh_revolute name="link_1_joint"
                      parent="base_link" child="link1"
                      a="${a1}" d="${d1}" alpha="${alpha1}"/>
-  <xacro:dh_revolute name="shoulder_lift_joint"
+  <!-- Joint 2: Shoulder Lift -->
+  <xacro:dh_revolute name="link_2_joint"
                      parent="link1" child="link2"
                      a="${a2}" d="${d2}" alpha="${alpha2}"/>
-  <xacro:dh_revolute name="elbow_joint"
+  <!-- Joint 3: Elbow -->
+  <xacro:dh_revolute name="link_3_joint"
                      parent="link2" child="link3"
                      a="${a3}" d="${d3}" alpha="${alpha3}"/>
-  <xacro:dh_revolute name="wrist_1_joint"
+  <!-- Joint 4: Wrist 1 -->
+  <xacro:dh_revolute name="link_4_joint"
                      parent="link3" child="link4"
                      a="${a4}" d="${d4}" alpha="${alpha4}"/>
-  <xacro:dh_revolute name="wrist_2_joint"
+  <!-- Joint 5: Wrist 2 -->
+  <xacro:dh_revolute name="link_5_joint"
                      parent="link4" child="link5"
                      a="${a5}" d="${d5}" alpha="${alpha5}"/>
-  <xacro:dh_revolute name="wrist_3_joint"
+  <!-- Joint 6: Wrist 3 -->
+  <xacro:dh_revolute name="link_6_joint"
                      parent="link5" child="link6"
                      a="${a6}" d="${d6}" alpha="${alpha6}"/>
-  <!-- Tool frame -->
+  <!-- Tool frame: end-effector reference point -->
   <link name="tool0"/>
   <joint name="tool0_fixed" type="fixed">
     <parent link="link6"/>
-    <child link="tool0"/>
+    <child  link="tool0"/>
     <origin xyz="0 0 0" rpy="0 0 0"/>
   </joint>
